File: Hardware/PCB Designs/PDB Board 0.2/PDB Board 0.2/PDB Board 0.2.kicad_pcb (KiCad board)
At the start: 4 copper layers, 50 x 50 mm, 54 parts, among them J1 ServoPort_06, J2 Conn_01x05, J3 Conn_01x05, J4 Conn_01x02, Q1 2N7002, U1 TPS62135RGXR, U2 IHLP2525CZER1R0M01, U3 AP2115R5-3.3TRG1

Commit message: PCB: add rev 0.3 PDB and MCU boards (female BtB sockets on MCU, PWM1 on PB4)
Parts:
- turned U2 to 0 degrees
Changed lines of the file:
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@@
 	(footprint "JLCImport:IHLP2525CZER1R0M01"
 		(layer "F.Cu")
-		(at 149.999872 96.5 180)
+		(at 149.999872 96.5)
 		(descr "11A 1uH 22A 7.6mΩ ±20% SMD,6.9x6.5mm Power Inductors ROHS")
 		(tags "C845018 IHLP2525CZER1R0M01 IND-SMD_L6.5-W6.5_IHLP-2525 Vishay Intertech")
@@
 		)
 		(property "Manufacturer" "Vishay Intertech"
-			(at 0 0 180)
+			(at 0 0 0)
 			(unlocked yes)
 			(layer "F.Fab")
@@
 		)
 		(property "Manufacturer Part" "IHLP2525CZER1R0M01"
-			(at 0 0 180)
+			(at 0 0 0)
 			(unlocked yes)
 			(layer "F.Fab")
@@
 		(duplicate_pad_numbers_are_jumpers no)
 		(fp_line
-			(start 3.25 3.25)
-			(end -3.25 3.25)
+			(start -3.25 -3.25)
+			(end 3.25 -3.25)
+			(stroke
+				(width 0.254)
+				(type solid)
+			)
+			(layer "F.SilkS")
+		)
+		(fp_line
+			(start -3.25 -1.946147)
+			(end -3.25 -3.25)
+			(stroke
+				(width 0.254)
+				(type solid)
+			)
+			(layer "F.SilkS")
+		)
+		(fp_line
+			(start -3.25 3.25)
+			(end -3.25 1.946147)
+			(stroke
+				(width 0.254)
+				(type solid)
+			)
+			(layer "F.SilkS")
+		)
+		(fp_line
+			(start 3.25 -3.25)
+			(end 3.25 -1.946147)
 			(stroke
 				(width 0.254)
@@
 		)
 		(fp_line
-			(start 3.25 -3.25)
-			(end 3.25 -1.946147)
-			(stroke
-				(width 0.254)
-				(type solid)
-			)
-			(layer "F.SilkS")
-		)
-		(fp_line
-			(start -3.25 3.25)
-			(end -3.25 1.946147)
-			(stroke
-				(width 0.254)
-				(type solid)
-			)
-			(layer "F.SilkS")
-		)
-		(fp_line
-			(start -3.25 -1.946147)
-			(end -3.25 -3.25)
-			(stroke
-				(width 0.254)
-				(type solid)
-			)
-			(layer "F.SilkS")
-		)
-		(fp_line
-			(start -3.25 -3.25)
-			(end 3.25 -3.25)
+			(start 3.25 3.25)
+			(end -3.25 3.25)
 			(stroke
 				(width 0.254)
@@
 		)
 		(pad "1" smd rect
-			(at -2.924505 0 180)
+			(at -2.924505 0)
 			(size 2.42 3.43)
 			(layers "F.Cu" "F.Mask" "F.Paste")
@@
 		)
 		(pad "2" smd rect
-			(at 2.924606 0 180)
+			(at 2.924606 0)
 			(size 2.42 3.43)
 			(layers "F.Cu" "F.Mask" "F.Paste")
